Commit message: added laser scanner

File: tortuga_description/urdf/tortuga_description.gazebo.urdf.xacro (robot description, xacro)
@@ -5,3 +5,6 @@
   <tortuga_motion/>
   <tortuga_xtion_plugin camera_name="camera"/>
+  <tortuga_hokuyo_macro name="laser" parent="base_footprint">
+      <origin xyz="0.05 0.0 0.36" rpy="0.0 0.0 0.0"/>
+  </tortuga_hokuyo_macro>
 </robot>

File: tortuga_description/urdf/tortuga_sensors.xacro (robot description, xacro)
@@ -53,3 +53,64 @@
       <link name="${name}_rgb_optical_frame"/>
   </xacro:macro>
+  <xacro:macro name="tortuga_hokuyo_macro" params="name parent *origin">
+    <joint name="${name}_joint" type="fixed">
+      <insert_block name="origin" />
+      <parent link="${parent}"/>
+      <child link="${name}"/>
+    </joint>
+    <link name="${name}">
+        <collision>
+        <origin xyz="0 0 0" rpy="0 0 0"/>
+        <geometry>
+        <box size="0.1 0.1 0.1"/>
+        </geometry>
+        </collision>
+        <visual>
+        <origin xyz="0 0 0" rpy="0 0 0"/>
+        <geometry>
+            <box size="0.05 0.05 0.05" /> <!-- does not need to match collision -->
+        </geometry>
+        </visual>
+        <inertial>
+        <mass value="1e-5" />
+        <origin xyz="0 0 0" rpy="0 0 0"/>
+        <inertia ixx="1e-6" ixy="0" ixz="0" iyy="1e-6" iyz="0" izz="1e-6" />
+        </inertial>
+    </link>
+      <gazebo reference="${name}">
+    <sensor type="gpu_ray" name="head_${name}_sensor">
+      <pose>0 0 0 0 0 0</pose>
+      <visualize>false</visualize>
+      <update_rate>40</update_rate>
+      <ray>
+        <scan>
+          <horizontal>
+            <samples>720</samples>
+            <resolution>1</resolution>
+            <min_angle>-1.570796</min_angle>
+            <max_angle>1.570796</max_angle>
+          </horizontal>
+        </scan>
+        <range>
+          <min>0.10</min>
+          <max>30.0</max>
+          <resolution>0.01</resolution>
+        </range>
+        <noise>
+          <type>gaussian</type>
+          <!-- Noise parameters based on published spec for Hokuyo laser
+               achieving "+-30mm" accuracy at range < 10m.  A mean of 0.0m and
+               stddev of 0.01m will put 99.7% of samples within 0.03m of the true
+               reading. -->
+          <mean>0.0</mean>
+          <stddev>0.01</stddev>
+        </noise>
+      </ray>
+      <plugin name="gazebo_ros_head_hokuyo_controller" filename="libgazebo_ros_gpu_laser.so">
+        <topicName>scan</topicName>
+        <frameName>${name}</frameName>
+      </plugin>
+    </sensor>
+  </gazebo>
+  </xacro:macro>
 </robot>
