Commit message: updated totuga sensor

File: tortuga_description/urdf/tortuga_sensors.xacro (robot description, xacro)
@@ -60,4 +60,5 @@
     </joint>
     <link name="${name}">
+        <!--
         <collision>
         <origin xyz="0 0 0" rpy="0 0 0"/>
@@ -69,7 +70,8 @@
         <origin xyz="0 0 0" rpy="0 0 0"/>
         <geometry>
-            <box size="0.05 0.05 0.05" /> <!-- does not need to match collision -->
+            <box size="0.05 0.05 0.05" />
         </geometry>
         </visual>
+        -->
         <inertial>
         <mass value="1e-5" />
@@ -81,5 +83,5 @@
     <sensor type="gpu_ray" name="head_${name}_sensor">
       <pose>0 0 0 0 0 0</pose>
-      <visualize>false</visualize>
+      <visualize>true</visualize>
       <update_rate>40</update_rate>
       <ray>
@@ -93,6 +95,6 @@
         </scan>
         <range>
-          <min>0.10</min>
-          <max>30.0</max>
+          <min>0.5</min>
+          <max>3.0</max>
           <resolution>0.01</resolution>
         </range>
